Commit message: added camera and lidar

File: src/diy_pkg/urdf/bot.xacro (robot description, xacro)
@@ -22,4 +22,11 @@
     <!-- BASE LINK -->
     <link name="base_link">
+    </link>
+    <joint name="base_footprint_joint" type="fixed">
+        <parent link="base_link"/>
+        <child link="base_footprint"/>
+        <origin xyz="0 0 0" rpy="0 0 0"/>
+    </joint>
+    <link name="base_footprint">
     </link>
     <!-- CHASSIS LINK -->
@@ -54,5 +61,5 @@
         <parent link="base_link"/>
         <child link="left_wheel"/>
-        <origin xyz="0 0.175 0" rpy="-${pi/2} 0 0" />
+        <origin xyz="0 0.175 0" rpy="-1.570796327 0 0" />
         <axis xyz="0 0 1"/>
     </joint>

File: src/diy_pkg/urdf/lidar.xacro (robot description, xacro)
@@ -29,5 +29,5 @@
         <sensor name="laser" type="ray">
             <pose>0 0 0 0 0 0</pose>
-            <visualize>false</visualize>
+            <visualize>true</visualize>
             <update_rate>10</update_rate>
             <ray>
